File: KiCAD files/generic module KiCAD/Stacked desk light.kicad_pcb (KiCad board)
At the start: 2 copper layers, 53.3 x 16.6 mm, 4 parts

Commit message: All new versions of generic and power boards
Parts:
- H1, H2: value Hex_Conn -> Hex_Conn_v2; footprint Stacked desk light:Conn_hex -> Stacked desk light:Conn_hex_v2
- turned D1 to 180 degrees
Connections:
- D1 pad 1: Net-(D1-Pad1) -> GND
- D1 pad 2: GND -> Net-(D1-Pad2)
- H1 pad 4: +5V -> GND
- H1 pad 5: +5V -> GND
- H1 pad 6: +5V -> GND
- H2 pad 4: +5V -> GND
- H2 pad 5: +5V -> GND
- H2 pad 6: +5V -> GND
- R1 pad 1: Net-(D1-Pad1) -> Net-(D1-Pad2)
Routing:
- net Net-(D1-Pad2): track 0.00 -> 6.46 mm
- net Net-(D1-Pad1): track 6.46 -> 0.00 mm
- net +5V: track 19.2 -> 23.2 mm
