File: KiCAD files/generic module KiCAD/Stacked desk light.sch (KiCad schematic (older format))
At the start: 4 parts

Commit message: All new versions of generic and power boards
Parts:
- removed H1, H2: Hex_Conn, Stacked desk light:Conn_hex, symbol Stacked~desk~light:Hex_Conn
- added H1, H2: Hex_Conn_v2, Stacked desk light:Conn_hex_v2, symbol Stacked~desk~light:Hex_Conn_v2
Connections:
- wire segments 0 -> 10
Other:
- moved on the sheet: D1
Changed lines of the file:
@@
 F 3 "~" H 3300 1700 50  0001 C CNN
 	1    3300 1700
-	0    1    1    0
+	0    -1   -1   0
 $EndComp
 $Comp
@@
 $EndComp
 $Comp
-L Stacked~desk~light:Hex_Conn H1
-U 1 1 60265E79
-P 2700 1350
-F 0 "H1" H 2662 1575 50  0000 C CNN
-F 1 "Hex_Conn" H 2662 1484 50  0000 C CNN
-F 2 "Stacked desk light:Conn_hex" H 2720 1615 50  0001 C CNN
-F 3 "" H 2700 1530 50  0001 C CNN
-	1    2700 1350
-	1    0    0    -1
-$EndComp
-$Comp
-L power:+5V #PWR0102
-U 1 1 6026CCAE
-P 2800 1650
-F 0 "#PWR0102" H 2800 1500 50  0001 C CNN
-F 1 "+5V" V 2815 1778 50  0000 L CNN
-F 2 "" H 2800 1650 50  0001 C CNN
-F 3 "" H 2800 1650 50  0001 C CNN
-	1    2800 1650
-	0    1    1    0
-$EndComp
-$Comp
-L power:+5V #PWR0103
-U 1 1 6026D23B
-P 2800 1750
-F 0 "#PWR0103" H 2800 1600 50  0001 C CNN
-F 1 "+5V" V 2815 1878 50  0000 L CNN
-F 2 "" H 2800 1750 50  0001 C CNN
-F 3 "" H 2800 1750 50  0001 C CNN
-	1    2800 1750
-	0    1    1    0
-$EndComp
-$Comp
 L power:+5V #PWR0104
 U 1 1 6026D38A
-P 2800 1850
-F 0 "#PWR0104" H 2800 1700 50  0001 C CNN
-F 1 "+5V" V 2815 1978 50  0000 L CNN
-F 2 "" H 2800 1850 50  0001 C CNN
-F 3 "" H 2800 1850 50  0001 C CNN
-	1    2800 1850
+P 2250 1900
+F 0 "#PWR0104" H 2250 1750 50  0001 C CNN
+F 1 "+5V" V 2265 2028 50  0000 L CNN
+F 2 "" H 2250 1900 50  0001 C CNN
+F 3 "" H 2250 1900 50  0001 C CNN
+	1    2250 1900
 	0    1    1    0
 $EndComp
@@
 L power:GND #PWR0107
 U 1 1 6026E472
-P 2800 1350
-F 0 "#PWR0107" H 2800 1100 50  0001 C CNN
-F 1 "GND" V 2805 1222 50  0000 R CNN
-F 2 "" H 2800 1350 50  0001 C CNN
-F 3 "" H 2800 1350 50  0001 C CNN
-	1    2800 1350
+P 2250 1300
+F 0 "#PWR0107" H 2250 1050 50  0001 C CNN
+F 1 "GND" V 2255 1172 50  0000 R CNN
+F 2 "" H 2250 1300 50  0001 C CNN
+F 3 "" H 2250 1300 50  0001 C CNN
+	1    2250 1300
 	0    -1   -1   0
 $EndComp
 $Comp
-L power:GND #PWR0108
-U 1 1 6026E7A1
-P 2800 1450
-F 0 "#PWR0108" H 2800 1200 50  0001 C CNN
-F 1 "GND" V 2805 1322 50  0000 R CNN
-F 2 "" H 2800 1450 50  0001 C CNN
-F 3 "" H 2800 1450 50  0001 C CNN
-	1    2800 1450
+L Stacked~desk~light:Hex_Conn_v2 H1
+U 1 1 608EFBC0
+P 2150 1300
+F 0 "H1" H 2112 1525 50  0000 C CNN
+F 1 "Hex_Conn_v2" H 2112 1434 50  0000 C CNN
+F 2 "Stacked desk light:Conn_hex_v2" H 2170 1565 50  0001 C CNN
+F 3 "" H 2150 1480 50  0001 C CNN
+	1    2150 1300
+	1    0    0    -1
+$EndComp
+Wire Wire Line
+	2250 1300 2250 1400
+Connection ~ 2250 1400
+Wire Wire Line
+	2250 1400 2250 1500
+Connection ~ 2250 1500
+Wire Wire Line
+	2250 1500 2250 1600
+Connection ~ 2250 1600
+Wire Wire Line
+	2250 1600 2250 1700
+Connection ~ 2250 1700
+Wire Wire Line
+	2250 1700 2250 1800
+Connection ~ 2250 1300
+$Comp
+L power:+5V #PWR0101
+U 1 1 608F994D
+P 2250 2900
+F 0 "#PWR0101" H 2250 2750 50  0001 C CNN
+F 1 "+5V" V 2265 3028 50  0000 L CNN
+F 2 "" H 2250 2900 50  0001 C CNN
+F 3 "" H 2250 2900 50  0001 C CNN
+	1    2250 2900
+	0    1    1    0
+$EndComp
+$Comp
+L power:GND #PWR0102
+U 1 1 608F9953
+P 2250 2300
+F 0 "#PWR0102" H 2250 2050 50  0001 C CNN
+F 1 "GND" V 2255 2172 50  0000 R CNN
+F 2 "" H 2250 2300 50  0001 C CNN
+F 3 "" H 2250 2300 50  0001 C CNN
+	1    2250 2300
 	0    -1   -1   0
 $EndComp
 $Comp
-L power:GND #PWR0109
-U 1 1 6026E9C7
-P 2800 1550
-F 0 "#PWR0109" H 2800 1300 50  0001 C CNN
-F 1 "GND" V 2805 1422 50  0000 R CNN
-F 2 "" H 2800 1550 50  0001 C CNN
-F 3 "" H 2800 1550 50  0001 C CNN
-	1    2800 1550
-	0    -1   -1   0
-$EndComp
-$Comp
-L Stacked~desk~light:Hex_Conn H2
-U 1 1 602753EA
-P 2700 2200
-F 0 "H2" H 2662 2425 50  0000 C CNN
-F 1 "Hex_Conn" H 2662 2334 50  0000 C CNN
-F 2 "Stacked desk light:Conn_hex" H 2720 2465 50  0001 C CNN
-F 3 "" H 2700 2380 50  0001 C CNN
-	1    2700 2200
+L Stacked~desk~light:Hex_Conn_v2 H2
+U 1 1 608F9959
+P 2150 2300
+F 0 "H2" H 2112 2525 50  0000 C CNN
+F 1 "Hex_Conn_v2" H 2112 2434 50  0000 C CNN
+F 2 "Stacked desk light:Conn_hex_v2" H 2170 2565 50  0001 C CNN
+F 3 "" H 2150 2480 50  0001 C CNN
+	1    2150 2300
 	1    0    0    -1
 $EndComp
-$Comp
-L power:+5V #PWR0110
-U 1 1 602753F0
-P 2800 2500
-F 0 "#PWR0110" H 2800 2350 50  0001 C CNN
-F 1 "+5V" V 2815 2628 50  0000 L CNN
-F 2 "" H 2800 2500 50  0001 C CNN
-F 3 "" H 2800 2500 50  0001 C CNN
-	1    2800 2500
-	0    1    1    0
-$EndComp
-$Comp
-L power:+5V #PWR0111
-U 1 1 602753F6
-P 2800 2600
-F 0 "#PWR0111" H 2800 2450 50  0001 C CNN
-F 1 "+5V" V 2815 2728 50  0000 L CNN
-F 2 "" H 2800 2600 50  0001 C CNN
-F 3 "" H 2800 2600 50  0001 C CNN
-	1    2800 2600
-	0    1    1    0
-$EndComp
-$Comp
-L power:+5V #PWR0112
-U 1 1 602753FC
-P 2800 2700
-F 0 "#PWR0112" H 2800 2550 50  0001 C CNN
-F 1 "+5V" V 2815 2828 50  0000 L CNN
-F 2 "" H 2800 2700 50  0001 C CNN
-F 3 "" H 2800 2700 50  0001 C CNN
-	1    2800 2700
-	0    1    1    0
-$EndComp
-$Comp
-L power:GND #PWR0113
-U 1 1 60275402
-P 2800 2200
-F 0 "#PWR0113" H 2800 1950 50  0001 C CNN
-F 1 "GND" V 2805 2072 50  0000 R CNN
-F 2 "" H 2800 2200 50  0001 C CNN
-F 3 "" H 2800 2200 50  0001 C CNN
-	1    2800 2200
-	0    -1   -1   0
-$EndComp
-$Comp
-L power:GND #PWR0114
-U 1 1 60275408
-P 2800 2300
-F 0 "#PWR0114" H 2800 2050 50  0001 C CNN
-F 1 "GND" V 2805 2172 50  0000 R CNN
-F 2 "" H 2800 2300 50  0001 C CNN
-F 3 "" H 2800 2300 50  0001 C CNN
-	1    2800 2300
-	0    -1   -1   0
-$EndComp
-$Comp
-L power:GND #PWR0115
-U 1 1 6027540E
-P 2800 2400
-F 0 "#PWR0115" H 2800 2150 50  0001 C CNN
-F 1 "GND" V 2805 2272 50  0000 R CNN
-F 2 "" H 2800 2400 50  0001 C CNN
-F 3 "" H 2800 2400 50  0001 C CNN
-	1    2800 2400
-	0    -1   -1   0
-$EndComp
+Wire Wire Line
+	2250 2300 2250 2400
+Connection ~ 2250 2400
+Wire Wire Line
+	2250 2400 2250 2500
+Connection ~ 2250 2500
+Wire Wire Line
+	2250 2500 2250 2600
+Connection ~ 2250 2600
+Wire Wire Line
+	2250 2600 2250 2700
+Connection ~ 2250 2700
+Wire Wire Line
+	2250 2700 2250 2800
+Connection ~ 2250 2300
 $EndSCHEMATC
