File: KiCAD files/power module KiCAD/Stacked desk light.kicad_pcb (KiCad board)
At the start: 2 copper layers, 53.3 x 16.6 mm, 6 parts, among them J1 USB_B_Micro, SW1 SW_DIP_x01

Commit message: All new versions of generic and power boards
Parts:
- added F1: Fuse_Small, Fuse:Fuse_0805_2012Metric_Pad1.15x1.40mm_HandSolder, F.Cu at (98.7, 96.6)
- H1, H2: value Hex_Conn -> Hex_Conn_v2; footprint Stacked desk light:Conn_hex -> Stacked desk light:Conn_hex_v2
- turned D1 to 180 degrees
Connections:
- D1 pad 1: Net-(D1-Pad1) -> GND
- D1 pad 2: GND -> Net-(D1-Pad2)
- H1 pad 4: +5V -> GND
- H1 pad 5: +5V -> GND
- H1 pad 6: +5V -> GND
- H2 pad 4: +5V -> GND
- H2 pad 5: +5V -> GND
- H2 pad 6: +5V -> GND
- J1 pad 1: Net-(J1-Pad1) -> Net-(F1-Pad2)
- R1 pad 1: Net-(D1-Pad1) -> Net-(D1-Pad2)
- SW1 pad 1: Net-(J1-Pad1) -> Net-(F1-Pad1)
Routing:
- net Net-(J1-Pad1): track 18.5 -> 0.00 mm
- net Net-(F1-Pad1): track 0.00 -> 11.6 mm
- net Net-(D1-Pad2): track 0.00 -> 6.46 mm
- net Net-(D1-Pad1): track 6.46 -> 0.00 mm
- net Net-(F1-Pad2): track 0.00 -> 4.80 mm
- net +5V: track 19.3 -> 23.0 mm
