File: KiCAD files/power module KiCAD/Stacked desk light.sch (KiCad schematic (older format))
At the start: 6 parts, among them J1 USB_B_Micro, SW1 SW_DIP_x01

Commit message: All new versions of generic and power boards
Parts:
- removed H1, H2: Hex_Conn, Stacked desk light:Conn_hex, symbol Stacked~desk~light:Hex_Conn
- added F1: Fuse_Small, Fuse:Fuse_0805_2012Metric_Pad1.15x1.40mm_HandSolder, symbol Device:Fuse_Small
- added H1, H2: Hex_Conn_v2, Stacked desk light:Conn_hex_v2, symbol Stacked~desk~light:Hex_Conn_v2
Connections:
- wire segments 3 -> 17
Other:
- moved on the sheet: D1, J1, R1, SW1
